Commit message: Tried with single elements on publisher, not a vector

File: src/ass_2/urdf/robot5.xacro (robot description, xacro)
@@ -104,4 +104,10 @@
 		<origin xyz="-0.1 -0.1 0"/>
 	</joint>
+   	 <joint name="camera_joint" type="fixed">
+	    <axis xyz="0 1 0" />
+	    <origin xyz="0.125 0 0.125" rpy="0 0 0"/>
+	    <parent link="base_link"/>
+	    <child link="camera_link"/>
+	  </joint>
         <!-- Camera -->
 	  <link name="camera_link">
@@ -127,10 +133,4 @@
 	    </inertial>
 	  </link>
-    	 <joint name="camera_joint" type="fixed">
-	    <axis xyz="0 1 0" />
-	    <origin xyz="0.125 0 0.125" rpy="0 0 0"/>
-	    <parent link="base_link"/>
-	    <child link="camera_link"/>
-	  </joint>
 	<!-- Planar move -->
 	<gazebo>
