Commit message: Created world

File: src/ass_2/urdf/robot.xacro (robot description, xacro)
@@ -1,5 +1,5 @@
 <?xml version="1.0"?>
-<robot xmlns:xacro="http://www.ros.org/wiki/xacro" name="robot5_xacro">
-<xacro:include filename="$(find ass_1)/urdf/robot5.gazebo"/>
+<robot xmlns:xacro="http://www.ros.org/wiki/xacro" name="robot_xacro">
+<xacro:include filename="$(find ass_2)/urdf/robot.gazebo"/>
 	<xacro:property name="length_wheel" value="0.05" />
 	<xacro:property name="radius_wheel" value="0.05" />
@@ -104,33 +104,4 @@
 		<origin xyz="-0.1 -0.1 0"/>
 	</joint>
-   	 <joint name="camera_joint" type="fixed">
-	    <axis xyz="0 1 0" />
-	    <origin xyz="0.125 0 0.125" rpy="0 0 0"/>
-	    <parent link="base_link"/>
-	    <child link="camera_link"/>
-	  </joint>
-        <!-- Camera -->
-	  <link name="camera_link">
-	    <collision>
-	      <origin xyz="0 0 0" rpy="0 0 0"/>
-	      <geometry>
-		<box size="0.05 0.05 0.05"/>
-	      </geometry>
-	    </collision>
-	    <visual>
-	      <origin xyz="0 0 0" rpy="0 0 0"/>
-	      <geometry>
-		<box size="0.05 0.05 0.05"/>
-	      </geometry>
-	      <material name="red">
-		<color rgba="1 0 0 1"/>
-	      </material>
-	    </visual>
-	    <inertial>
-	      <mass value="1e-5" />
-	      <origin xyz="0 0 0" rpy="0 0 0"/>
-	      <inertia ixx="1e-6" ixy="0" ixz="0" iyy="1e-6" iyz="0" izz="1e-6" />
-	    </inertial>
-	  </link>
 	<!-- Planar move -->
 	<gazebo>

Commit message: Uploaded simulation in gazebo

File: src/ass_2/urdf/robot.xacro (robot description, xacro)
@@ -22,5 +22,5 @@
        				<box size="0.2 .3 .1"/>
      			</geometry>
-			<origin rpy="0 0 0" xyz="0 0 0.05"/>
+			<origin rpy="0 0 1.5707" xyz="0 0 0.05"/>
 			<material name="white">
 				<color rgba="1 1 1 1"/>
@@ -37,5 +37,5 @@
    		<visual>
      			<xacro:wheel_geometry />
-			<origin rpy="0 1.5707 0" xyz="0.0 0.0 0"/>
+			<origin rpy="0 1.5707 1.5707" xyz="0.0 0.0 0"/>
    			<material name="black">
 				<color rgba="0 0 0 1"/>
@@ -50,5 +50,5 @@
    		<visual>
      			<xacro:wheel_geometry />
-			<origin rpy="0 1.5707 0" xyz="-0.0 0.0 0"/>
+			<origin rpy="0 1.5707 1.5707" xyz="-0.0 0.0 0"/>
    			<material name="black"/>
    		</visual>
@@ -61,5 +61,5 @@
    		<visual>
  			<xacro:wheel_geometry />
-			<origin rpy="0 1.5707 0" xyz="0.0 -0.0 0"/>
+			<origin rpy="0 1.5707 1.5707" xyz="0.0 -0.0 0"/>
    			<material name="black"/>
    		</visual>
@@ -72,5 +72,5 @@
    		<visual>
   			 <xacro:wheel_geometry />
-			<origin rpy="0 1.5707 0" xyz="-0.0 -0.0 0"/>
+			<origin rpy="0 1.5707 1.5707" xyz="-0.0 -0.0 0"/>
    			<material name="black"/>
    		</visual>

Commit message: Now it works in all the cases

File: src/ass_2/urdf/robot.xacro (robot description, xacro)
@@ -22,5 +22,5 @@
        				<box size="0.2 .3 .1"/>
      			</geometry>
-			<origin rpy="0 0 1.5707" xyz="0 0 0.05"/>
+			<origin rpy="0 0 1.5707" xyz="0 0 0.05"/> <!-- 1.5707 -->
 			<material name="white">
 				<color rgba="1 1 1 1"/>
